File: To_the_moon.sch (KiCad schematic (older format))
At the start: 13 parts, among them J1 USB_C_Receptacle_USB2.0, U1 HW-755, U2 2.4_tft_display, U3 WeMos_D1_mini

Commit message: Added kicad main files
Parts:
- removed D1: WS2812, LED_SMD:LED_WS2812_PLCC6_5.0x5.0mm_P1.6mm, symbol LED:WS2812
- removed J1: USB_C_Receptacle_USB2.0, symbol Connector:USB_C_Receptacle_USB2.0
- removed RESET1: SW_Push, symbol Switch:SW_Push
- removed U1: HW-755, symbol Power_Management:HW-755
- removed U2: 2.4_tft_display, symbol Display_Graphic:wemos_2.4_tft_display
- removed U3: WeMos_D1_mini, Module:WEMOS_D1_mini_light, symbol MCU_Module:WeMos_D1_mini
- added C10, C8: 10uf, Capacitor_SMD:C_0603_1608Metric, symbol Device:C_Small
- added C11, C14: 4.7uf, Capacitor_SMD:C_1206_3216Metric, symbol Device:C_Small
- added C12, C13: 1uf, Capacitor_SMD:C_0603_1608Metric, symbol Device:C_Small
- added C6: 100uf, Capacitor_SMD:C_1206_3216Metric, symbol Device:C_Small
- added C7, C9: 0.1uf, Capacitor_SMD:C_0603_1608Metric, symbol Device:C_Small
- added D1, D5: Blue, LED_SMD:LED_0805_2012Metric, symbol Device:LED_Small
- added D3, D6: Yellow, LED_SMD:LED_0805_2012Metric, symbol Device:LED_Small
- added D4: WS2812B, LED_SMD:WS2812-2020, symbol LED:WS2812B
- added D7: D_Schottky, Diode_SMD:D_SOD-123, symbol Device:D_Schottky
- added H1, H2, H3, H4: MountingHole, MountingHole:MountingHole_3.2mm_M3_DIN965_Pad, symbol Mechanical:MountingHole
- added H6: MountingHole, MountingHole:MountingHole_2.1mm, symbol Mechanical:MountingHole
- added IC1: DW01A, Package_TO_SOT_SMD:SOT-23-6, symbol Power_Protection:DW01A
- added J1: USB_B_Micro, Connector_USB:USB_Micro-B_Molex-105017-0001, symbol Connector:USB_B_Micro
- added J2: connector lipo, Connector_PinHeader_2.00mm:PinHeader_1x02_P2.00mm_Vertical, symbol Connector:Conn_01x02_Female
- added J3: Conn_01x09_Male, Connector_PinHeader_2.00mm:PinHeader_1x09_P2.00mm_Vertical, symbol Connector:Conn_01x09_Male
- added J4: Conn_01x03_Female, Connector_PinHeader_2.00mm:PinHeader_1x03_P2.00mm_Vertical_SMD_Pin1Left, symbol Connector:Conn_01x03_Female
- added L1: 10uh, Inductor_SMD:L_1206_3216Metric, symbol pspice:INDUCTOR
- added Q1: FS8205, Package_TO_SOT_SMD:SOT-23-6, symbol Transistor_Array:FS8205
- added Q2, Q3: BC847, Package_TO_SOT_SMD:SOT-23, symbol Transistor_BJT:BC847
- added Q4: AO3401A, Package_TO_SOT_SMD:SOT-23, symbol Transistor_FET:AO3401A
- added R10, R7: 470, Resistor_SMD:R_0603_1608Metric, symbol Device:R_Small
- added R11: 100, Resistor_SMD:R_0603_1608Metric, symbol Device:R_Small
- added R12, R13: 2K, Resistor_SMD:R_0603_1608Metric, symbol Device:R_Small
- added R14, R18, R4, R8, R9: 10K, Resistor_SMD:R_0603_1608Metric, symbol Device:R_Small
- added R15: 100K, Resistor_SMD:R_0603_1608Metric, symbol Device:R_Small
- added R16: 62K, Resistor_SMD:R_0603_1608Metric, symbol Device:R_Small
- added R17: 8.2K, Resistor_SMD:R_0603_1608Metric, symbol Device:R_Small
- added R3, R5: 1.2K, Resistor_SMD:R_0603_1608Metric, symbol Device:R_Small
- added R6: 1K, Resistor_SMD:R_0603_1608Metric, symbol Device:R_Small
- added SW1, SW2: SW_Push, Button_Switch_SMD:TS-1187A-B-A-B, symbol Switch:SW_Push
- added U1: ESP-12E, RF_Module:ESP-12E, symbol RF_Module:ESP-12E
- added U2: TP4056, Package_SO:HSOP-8-1EP_3.9x4.9mm_P1.27mm_EP2.41x3.1mm, symbol Power_Management:TP4056
- added U3: CH340G, Package_SO:SOIC-16_3.9x9.9mm_P1.27mm, symbol Interface_USB:CH340G
- added U4: MT3608, Package_TO_SOT_SMD:SOT-23-6, symbol Regulator_Switching:MT3608
- added U5: AMS1117-3.3, Package_TO_SOT_SMD:SOT-223-3_TabPin2, symbol Regulator_Linear:AMS1117-3.3
- added Y1: 12MHz, Crystal:Crystal_SMD_TXC_7M-4Pin_3.2x2.5mm, symbol Device:Crystal_GND24_Small
- C1: value 15p -> 14pf; footprint (none) -> Capacitor_SMD:C_0402_1005Metric; LCSC (none) -> C458857
- C2: value 100 -> 14pf; footprint (none) -> Capacitor_SMD:C_0402_1005Metric; LCSC (none) -> C458857
- C3: value 10 -> 10uf; footprint (none) -> Capacitor_SMD:C_0603_1608Metric; LCSC (none) -> C19702
- C4: value 100 -> 10uf; footprint (none) -> Capacitor_SMD:C_0603_1608Metric; LCSC (none) -> C19702
- C5: value 10 -> 100uf; footprint (none) -> Capacitor_SMD:C_1206_3216Metric; LCSC (none) -> C15008
- R1: value 150 -> 1.2K; footprint (none) -> Resistor_SMD:R_0603_1608Metric; LCSC (none) -> C22765
- R2: value 10k -> 10K; footprint (none) -> Resistor_SMD:R_0603_1608Metric; LCSC (none) -> C25804
Connections:
- net labels added: 5VUSB, 5V_, D+, D-, D0, D3, D5, D6, D7, D8, DTR, EN, GND_, GPIO0, GPIO4, LED, LED_, OC, OD, RST, RTS, RX, TX, VCC, XI, XO
- net labels removed: +BATT, 5Vin, Data_LED, TFT_CS, TFT_DC, TS_CS
- wire segments 44 -> 167
Other:
- note added: "(14pfx14pf) / (14pf+14pf) + 5 = 12pf"
- note removed: "Power management"
- note removed: "WS2812 LED"

Commit message: Update PDF schematic
Parts:
- removed D4: WS2812B, LED_SMD:WS2812-2020, symbol LED:WS2812B
- added U6: WS2812-2020, LED_SMD:WS2812-2020, symbol LED:WS2812-2020
Connections:
- wire segments 167 -> 165
Other:
- note added: "3.3V regulator"
- note added: "5V regulator"
- note added: "Battery charger with load sharing"
- note added: "Breakout LCD"
- note added: "ESP8266"
- note added: "Pullup"
- note added: "Small breakout board LED"
- note added: "USB serial programmer"
- moved on the sheet: C1, C2, C4, C6, C9, R14, R18, R2, R4, SW1, SW2
